File: hardware/projects/MicBac/PROJ-FRL-RIFD_Box/Electro/FRL-RFiD_Box/FRL-RFiD_Box.kicad_pcb (KiCad board)
At the start: 2 copper layers, 100 x 72 mm, 38 parts, among them J1 I2C_OLED, J2 SPI_NFC, J3 WAGO OTHER, J4 WAGO (230V), J5 USB_C_Receptacle, K1 FINDER-41.52.9.024.4311, Q1 IRLZ44N, Q2 BC547, Q3 DMG2305UX, U1 RAC05-24SK, U2 R-78C5.0-1.0, U4 ESP32-S3-WROOM-1, U5 PC817, U6 AMS1117-3.3

Commit message: Kicad-Add PN532 (NFC), Change Schematic Power, PCB arrange Power
Parts:
- removed C1, C2: 10u 50V MLCC, Capacitor_SMD:C_1206_3216Metric
- removed J4: WAGO (230V), TerminalBlock_WAGO:TerminalBlock_WAGO_2601-1104_1x04_P3.50mm_Horizontal
- removed L1: 12u choke RLS-126, Inductor_SMD:L_1812_4532Metric
- removed U2: R-78C5.0-1.0, Converter_DCDC:Converter_DCDC_RECOM_R-78E-0.5_THT
- added C15: 1u, Capacitor_SMD:C_0603_1608Metric, F.Cu at (95.0, 152.8)
- added C16: 10u, Capacitor_SMD:C_0603_1608Metric, F.Cu at (52.5, 153.3)
- added C17: 100n, Capacitor_SMD:C_0603_1608Metric, F.Cu at (52.5, 155.8)
- added C18: 100n, Capacitor_SMD:C_0603_1608Metric, F.Cu at (52.5, 158.3)
- added C19: 10u, Capacitor_SMD:C_0603_1608Metric, F.Cu at (52.5, 160.8)
- added C20: 100n, Capacitor_SMD:C_0603_1608Metric, F.Cu at (52.5, 163.3)
- added C21: 100n, Capacitor_SMD:C_0603_1608Metric, F.Cu at (52.5, 165.8)
- added C22: 4,7u, Capacitor_SMD:C_0603_1608Metric, F.Cu at (52.5, 168.3)
- added C23: 22p, Capacitor_SMD:C_0603_1608Metric, F.Cu at (52.5, 170.8)
- added C24: 22p, Capacitor_SMD:C_0603_1608Metric, F.Cu at (52.5, 173.3)
- added C4: 10u, Capacitor_SMD:C_0603_1608Metric, F.Cu at (189.8, 101.2)
- added D6: SMAJ36CA, Diode_SMD:D_SMA, F.Cu at (205.8, 120.6)
- added D7: LED G, LED_SMD:LED_0603_1608Metric, F.Cu at (209.3, 114.6)
- added D8: ESD9B3.3ST5G, Diode_SMD:D_SOD-923, F.Cu at (98.4, 152.5)
- added F1: 200mA T, Fuse:Fuse_Schurter_UMZ250, F.Cu at (200.8, 120.6)
- added J10: Conn_01x05, Connector_PinHeader_2.54mm:PinHeader_1x05_P2.54mm_Vertical, B.Cu at (70.0, 115.0)
- added J11: Conn_02x02_Odd_Even, Connector_PinHeader_2.54mm:PinHeader_2x02_P2.54mm_Vertical, F.Cu at (168.7, 123.7)
- added J12: Conn_02x02_Odd_Even, Connector_PinHeader_2.54mm:PinHeader_2x02_P2.54mm_Vertical, F.Cu at (248.7, 123.7)
- added J13: Conn_02x02_Odd_Even, Connector_PinHeader_2.54mm:PinHeader_2x02_P2.54mm_Vertical, B.Cu at (61.3, 63.7)
- added J14: Conn_02x02_Odd_Even, Connector_PinHeader_2.54mm:PinHeader_2x02_P2.54mm_Vertical, B.Cu at (61.3, 123.7)
- added J15: Conn_02x02_Odd_Even, Connector_PinHeader_2.54mm:PinHeader_2x02_P2.54mm_Vertical, B.Cu at (146.3, 63.7)
- added J16: Conn_02x02_Odd_Even, Connector_PinHeader_2.54mm:PinHeader_2x02_P2.54mm_Vertical, B.Cu at (146.3, 123.7)
- added J7: Conn_02x02_Odd_Even, Connector_PinHeader_2.54mm:PinHeader_2x02_P2.54mm_Vertical, F.Cu at (168.7, 63.7)
- added J8: Conn_02x02_Odd_Even, Connector_PinHeader_2.54mm:PinHeader_2x02_P2.54mm_Vertical, F.Cu at (248.7, 63.7)
- added J9: Conn_01x05, Connector_PinHeader_2.54mm:PinHeader_1x05_P2.54mm_Vertical, F.Cu at (180.0, 115.0)
- added PS1: RS6-2405S, MOD-DC_DC_Converters:CONV_RS6-2405S, F.Cu at (207.3, 99.1)
- added R10: 10k, Resistor_SMD:R_0603_1608Metric, F.Cu at (95.0, 155.3)
- added R7: 22k, Resistor_SMD:R_0603_1608Metric, F.Cu at (189.8, 92.2)
- added R8: 2k2, Resistor_SMD:R_0603_1608Metric, F.Cu at (205.3, 114.6)
- added R9: 2k2, Resistor_SMD:R_0603_1608Metric, F.Cu at (207.3, 114.6)
- added U3: PN5321A3HN_C1xx, Package_DFN_QFN:HVQFN-40-1EP_6x6mm_P0.5mm_EP4.1x4.1mm, F.Cu at (59.0, 156.2)
- added Y1: 27.12MHz, PCM_SparkFun-Clock:Crystal_SMD_3.2x2.5mm, F.Cu at (56.9, 162.4)
- C9: value 1u -> 10u
- J3: value WAGO OTHER -> WAGO (230V + 24V)
- moved U1 167.3 mm to (238.3, 99.3), turned to 0 degrees
- moved R2 142.2 mm to (207.8, 85.6)
- moved K1 132.5 mm to (216.4, 67.3), turned to 0 degrees
- moved D1 122.6 mm to (210.3, 66.0), turned to -90 degrees
- moved Q1 111.1 mm to (204.8, 82.0), turned to 0 degrees
- moved U5 102.4 mm to (198.0, 69.8), turned to 0 degrees
- moved J3 101.4 mm to (216.0, 119.1)
- moved Q3 89.5 mm to (193.8, 96.7), turned to 0 degrees
- moved R3 86.7 mm to (194.8, 70.1), turned to 0 degrees
- moved C14 85.4 mm to (197.3, 110.3)
- moved C13 85.4 mm to (193.3, 110.3)
- moved U6 85.4 mm to (195.3, 104.2)
- moved C3 85.3 mm to (197.8, 96.0), turned to 90 degrees
- moved D5 85.1 mm to (189.8, 96.7), turned to 90 degrees
- moved C8 82.0 mm to (63.9, 106.5), turned to 180 degrees
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Connections:
- net /+5V_R-78C5.0_OUT renamed /+5V_RS6-2405S_+VOUT
- C13 pad 1: +3V3 -> +3V3 Bot
- C14 pad 1: +3V3 -> +3V3 Bot
- D5 pad 1: +5V -> +5V Bot
- D5 pad 2: /VBUS -> /VBUS Bot
- J3 pad 1: unconnected-(J3-Pin_1-Pad1) -> 24_GND
- J3 pad 2: unconnected-(J3-Pin_2-Pad2) -> /+24V_RAC05_OUT
- J3 pad 4: unconnected-(J3-Pin_4-Pad4) -> /230V_AC_FINDER_N (OUT)
- J3 pad 5: unconnected-(J3-Pin_5-Pad5) -> /230V_AC_FINDER_L (OUT)
- J3 pad 7: unconnected-(J3-Pin_7-Pad7) -> /230V_AC_RAC05_L (IN)
- J3 pad 8: unconnected-(J3-Pin_8-Pad8) -> /230V_AC_RAC05_N (IN)
- Q1 pad 3: GND -> 24_GND
- Q3 pad 1: /VBUS -> /VBUS Bot
- Q3 pad 2: +5V -> +5V Bot
- R2 pad 2: GND -> 24_GND
- R3 pad 1: /PC817 (OPT) -> /PC817 (OPT) Bot
- U1 pad 4: GND -> 24_GND
- U4 pad 26: /BUZZER -> unconnected-(U4-IO45-Pad26)
- U4 pad 27: unconnected-(U4-IO0-Pad27) -> /ESP_IO_0
- U4 pad 33: unconnected-(U4-IO40-Pad33) -> /BUZZER
- U4 pad 36: unconnected-(U4-RXD0-Pad36) -> /ESP_RXD
- U4 pad 37: unconnected-(U4-TXD0-Pad37) -> /ESP_TXD
- U6 pad 2: +3V3 -> +3V3 Bot
- U6 pad 3: +5V -> +5V Bot
Routing:
- net /+24V_RAC05_OUT: track 0.00 -> 94.7 mm
- net /230V_AC_FINDER_N (OUT): track 0.00 -> 67.7 mm
- net /230V_AC_RAC05_N (IN): track 0.00 -> 58.5 mm
- net /PC817 (OPT) Bot: track 0.00 -> 54.8 mm
- net /230V_AC_RAC05_L (IN): track 0.00 -> 47.5 mm
- net /230V_AC_FINDER_L (OUT): track 0.00 -> 46.9 mm
- net +5V Bot: track 0.00 -> 37.0 mm
- net +3V3 Bot: track 0.00 -> 34.8 mm
- net /VBUS Bot: track 0.00 -> 34.2 mm
- net /+24V_RS6_+VIN: track 0.00 -> 34.1 mm
- net +3V3: track 0.00 -> 22.5 mm
- net /+5V_RS6-2405S_+VOUT: track 0.00 -> 16.5 mm
- net Net-(Q1-G): track 0.00 -> 15.2 mm
- net Net-(D1-A): track 0.00 -> 13.8 mm
- net /PC817 (OPT): track 0.00 -> 12.7 mm
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Other:
- board size 100 x 72 mm -> 200 x 70 mm
