File: hardware/projects/MicBac/PROJ-FRL-RIFD_Box/Electro/FRL-RFiD_Box/FRL-RFiD_Box.kicad_sch (KiCad schematic)
At the start: 40 parts, among them J1 I2C_OLED, J2 SPI_NFC, J3 WAGO OTHER, J4 WAGO (230V), J5 USB_C_Receptacle, K1 FINDER-41.52.9.024.4311, Q1 IRLZ44N, Q2 BC547, Q3 DMG2305UX, U1 RAC05-24SK, U2 R-78C5.0-1.0, U4 ESP32-S3-WROOM-1, U5 PC817, U6 AMS1117-3.3

Commit message: Kicad-Add PN532 (NFC), Change Schematic Power, PCB arrange Power
Parts:
- removed C1, C2: 10u 50V MLCC, Capacitor_SMD:C_1206_3216Metric, symbol Device:C_Small
- removed U2: R-78C5.0-1.0, Converter_DCDC:Converter_DCDC_RECOM_R-78E-0.5_THT, symbol Converter_DCDC:R-78C5.0-1.0
- added C15: 1u, Capacitor_SMD:C_0603_1608Metric, symbol Device:C_Small
- added C16, C19: 10u, Capacitor_SMD:C_0603_1608Metric, symbol Device:C_Small
- added C17, C18, C20, C21, C32, C33: 100n, Capacitor_SMD:C_0603_1608Metric, symbol Device:C_Small
- added C22: 4,7u, Capacitor_SMD:C_0603_1608Metric, symbol Device:C_Small
- added C23, C24, C26, C29: 22p, Capacitor_SMD:C_0603_1608Metric, symbol Device:C_Small
- added C25, C28: 220p, Capacitor_SMD:C_0603_1608Metric, symbol Device:C_Small
- added C27, C30: 200p, Capacitor_SMD:C_0603_1608Metric, symbol Device:C_Small
- added C31: 1n, Capacitor_SMD:C_0603_1608Metric, symbol Device:C_Small
- added D6: SMAJ36CA, Diode_SMD:D_SMA, symbol Diode:SMAJ36CA
- added D7: LED G, LED_SMD:LED_0603_1608Metric, symbol Device:LED
- added D8: ESD9B3.3ST5G, Diode_SMD:D_SOD-923, symbol Diode:ESD9B3.3ST5G
- added F1: 200mA T, Fuse:Fuse_Schurter_UMZ250, symbol Device:Fuse_Small
- added J10, J9: Conn_01x05, Connector_PinHeader_2.54mm:PinHeader_1x05_P2.54mm_Vertical, symbol Connector_Generic:Conn_01x05
- added J11, J12, J13, J14, J15, J16, J7, J8: Conn_02x02_Odd_Even, Connector_PinHeader_2.54mm:PinHeader_2x02_P2.54mm_Vertical, symbol Connector_Generic:Conn_02x02_Odd_Even
- added J6: Conn_02x03_Odd_Even, symbol Connector_Generic:Conn_02x03_Odd_Even
- added L2: 560m, symbol Device:L_Small
- added PS1: RS6-2405S, MOD-DC_DC_Converters:CONV_RS6-2405S, symbol RS6-2405S:RS6-2405S
- added R10: 10k, Resistor_SMD:R_0603_1608Metric, symbol Device:R_Small
- added R11, R12: 1.6k, Resistor_SMD:R_0603_1608Metric, symbol Device:R_Small
- added R8, R9: 2k2, Resistor_SMD:R_0603_1608Metric, symbol Device:R
- added SW1: SW_SPST, symbol Switch:SW_SPST
- added U3: PN5321A3HN_C1xx, Package_DFN_QFN:HVQFN-40-1EP_6x6mm_P0.5mm_EP4.1x4.1mm, symbol RF_NFC:PN5321A3HN_C1xx
- added Y1: 27.12MHz, PCM_SparkFun-Clock:Crystal_SMD_3.2x2.5mm, symbol PCM_SparkFun-Clock:Crystal_27.12MHz_3.2x2.5mm
- C9: value 1u -> 10u
- J3: value WAGO OTHER -> WAGO (230V + 24V)
- J4: value WAGO (230V) -> WAGO (OTHER); now left out of the parts list
- L1: value 12u choke RLS-126 -> 560m; footprint Inductor_SMD:L_1812_4532Metric -> (none)
- R7: footprint (none) -> Resistor_SMD:R_0603_1608Metric
Connections:
- net +24V_RAC05_OUT: now also J3.2 (Pin_2), D6.2 (A2), F1.1; no longer L1.1
- net +3V3: now also C17.1, C18.1, C19.1, C20.1, C21.1, C22.1, J10.4 (Pin_4), J6.2 (Pin_2), R10.2, U3.17 (I1), U3.23 (PVDD), U3.40 (VBAT), U3.5 (TVDD); no longer C13.1, C14.1, U6.2 (VO)
- net +5V: now also J10.3 (Pin_3); no longer C4.1, D5.1 (K), Q3.2 (S), U6.3 (VI)
- net 230V_AC_FINDER_L (OUT): now also J3.5 (Pin_5); no longer J4.3 (Pin_3)
- net 230V_AC_FINDER_N (OUT): now also J3.4 (Pin_4); no longer J4.4 (Pin_4)
- net 230V_AC_RAC05_L (IN): now also J3.7 (Pin_7); no longer J4.1 (Pin_1)
- net 230V_AC_RAC05_N (IN): now also J3.8 (Pin_8); no longer J4.2 (Pin_2)
- net BUZZER: now also U4.33 (IO40); no longer U4.26 (IO45)
- net EN: now also J6.1 (Pin_1)
- net GND: now also C15.2, C16.2, C17.2, C18.2, C19.2, C20.2, C21.2, C22.2, C23.2, C24.2, C25.2, C27.2, C28.1, C30.1, C32.2, C33.2, D8.1 (A1), J10.5 (Pin_5), J6.4 (Pin_4), J9.5 (Pin_5), PS1.7 (-VOUT), SW1.1 (A), U3.1 (DVSS), U3.11 (AVSS), U3.16 (I0), U3.18 (TESTEN), U3.3 (TVSS1), U3.41 (AVSS), U3.7 (TVSS2); no longer Q1.3 (S), R2.2, U1.4 (-Vout)
- net PC817 (OPT): now also J10.1 (Pin_1); no longer R3.1
- net SPI_NFC_IRQ: now also U3.25 (P70_IRQ)
- net SPI_NFC_MISO: now also U3.29 (MISO/P71)
- net SPI_NFC_MOSI: now also U3.28 (MOSI/SDA/HSU_TX)
- net SPI_NFC_SCK: now also U3.30 (SCK/P72)
- net SPI_NFC_SS: now also U3.27 (NSS/P50_SCL/HSU_RX)
- net VBUS: now also C16.1, J10.2 (Pin_2); no longer D5.2 (A), Q3.1 (G), R7.1
- net ESP_IO_0: now reaches U4.27 (IO0)
- net ESP_IO_0: now also C15.1, D8.2 (A2), J6.6 (Pin_6), R10.1, SW1.2 (B)
- net ESP_RXD: now reaches U4.36 (RXD0)
- net ESP_RXD: now also J6.5 (Pin_5)
- net ESP_TXD: now reaches U4.37 (TXD0)
- net ESP_TXD: now also J6.3 (Pin_3)
- net NFC_INT0_IRQ: now reaches U4.6 (IO6)
- net NFC_INT0_IRQ: now also U3.32 (P32_INT0)
- net NFC_nRSTPD: now reaches U4.7 (IO7)
- net NFC_nRSTPD: now also U3.38 (~{RSTPD})
- net 24_GND: now reaches J3.1 (Pin_1)
- net 24_GND: now also Q1.3 (S), R2.2, U1.4 (-Vout), D6.1 (A1), D7.1 (K), PS1.1 (-VIN)
- net +24V_R-78C5.0_IN: no longer names the net of L1.2
- net +24V_R-78C5.0_IN: now also C25.1, C26.2
- net +5V_R-78C5.0_OUT renamed +5V_RS6-2405S_+VOUT
- net +5V_RS6-2405S_+VOUT: now also PS1.6 (+VOUT)
- new net: C28.2, C29.2, L2.2, R11.1
- new net: C31.1, R11.2
- new net: C26.1, C27.1
- new net: C23.1, U3.14 (OSCIN), Y1.1
- new net: C33.1, U3.37 (SVDD)
- new net: C24.1, U3.15 (OSCOUT), Y1.2
- new net: L2.1, U3.6 (TX2)
- new net: C29.1, C30.2
- new net: C32.1, R12.2, U3.9 (VMID)
- new net: C31.2, R12.1, U3.10 (RX)
- new net: L1.1, U3.4 (TX1)
- new net: D7.2 (A), R9.2
- new net: R8.2, R9.1
- new net +24V_RS6_+VIN: F1.2, PS1.2 (+VIN), R8.1
- new net +3V3 Bot: C13.1, C14.1, J9.4 (Pin_4), U6.2 (VO)
- new net +5V Bot: C4.1, D5.1 (K), J9.3 (Pin_3), Q3.2 (S), U6.3 (VI)
- new net PC817 (OPT) Bot: J9.1 (Pin_1), R3.1
- new net VBUS Bot: D5.2 (A), J9.2 (Pin_2), Q3.1 (G), R7.1
- no-connect marks 4 -> 58
Other:
- note added: "Fuse: 3403.0159.24"
- moved on the sheet: BZ1, C10, C11, C12, C13, C14, C3, C4, C7, C8, C9, D1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
