File: hardware/projects/RFID_BOX/cad/PoC/PoC.kicad_sch (KiCad schematic)
At the start: 10 parts, among them J1 Screw_Terminal_01x03, J2 Screw_Terminal_01x03, K1 T92S11D12-24, U1 ESP32-S3-WROOM-1, U2 PN5321A3HN_C1xx, U3 IRM-10-24, U4 AMS1117-3.3

Commit message: progress
Parts:
- removed J1, J2: Screw_Terminal_01x03, symbol Connector:Screw_Terminal_01x03
- removed U3: IRM-10-24, Converter_ACDC:Converter_ACDC_MeanWell_IRM-10-xx_THT, symbol Converter_ACDC:IRM-10-24
- added J1, J2: J_WAGO_2604-1103, aa_MyParts:J_2604-1103_WAG, symbol aa_MyParts:J_WAGO_2604-1103
- added J3: F_696309001002, aa_MyParts:F_Wurth_WR-FSH_696309001002, symbol aa_MyParts:F_696309001002
- added K2: K_G5V-1-2_DC24, aa_MyParts:K_G5V-1-2_DC24, symbol aa_MyParts:K_G5V-1-2_DC24
- added LED1: LED_IN-PI20TATPRPGPB, aa_MyParts:LED_INPI20TATPRPGPB, symbol aa_MyParts:LED_IN-PI20TATPRPGPB
- added PS1: IC_R-78K5.0-2.0, aa_MyParts:IC_CONV_R-78K5.0-2.0, symbol aa_MyParts:IC_R-78K5.0-2.0
- added U3: IC_IRM-10-24, aa_MyParts:IC_IRM-10-24_THT, symbol aa_MyParts:IC_IRM-10-24
- added U5: IC_RFB-0505S, aa_MyParts:IC_RFB-0505S, symbol aa_MyParts:IC_RFB-0505S
- added U6: MCP39F511A-E/MQ, aa_MyParts:IC_QFN28_MQ_MCH, symbol aa_MyParts:IC_MCP39F511A-E_MQ
Connections:
- new net: J1.1 (Pin_1), J1.2 (Pin_2)
- new net: J1.3 (Pin_3), J1.4 (Pin_4)
- new net: J1.5 (Pin_5), J1.6 (Pin_6)
- new net: J2.1 (Pin_1), J2.2 (Pin_2)
- new net: J2.3 (Pin_3), J2.4 (Pin_4)
- new net: J2.5 (Pin_5), J2.6 (Pin_6)
- new net: K2.5, K2.6
Other:
- note removed: "696309001002"
- note removed: "G5V-1-2 DC24"
- note removed: "IN-PI20TATPRPGPB"
- note removed: "MCP39F51A"
- note removed: "R-78K5.0-2.0"
- note removed: "RFB-0505S"
