File: hardware/projects/RFID_BOX/ECAD/IO_Board/IO_Board.kicad_pcb (KiCad board)
At the start: 2 copper layers, 13 parts, among them J1 J_WAGO_2604-1103, J2 J_WAGO_2604-1103, J3 F_696309001002, K1 T92S11D12-24, K2 K_G5V-1-2_DC24, U1 ESP32-S3-WROOM-1, U2 PN5321A3HN_C1xx, U3 IC_IRM-10-24, U4 AMS1117-3.3, U5 IC_RFB-0505S, U6 MCP39F511A-E/MQ

Commit message: Konkretisiere EMV-Bauteile und NTC in BOM, verschiebe PoC-KiCad-Projekt nach ECAD/IO_Board
- EMV Maßnahmen in Bauteilauswahl auf MOV, X2-Kondensator und Gleichtaktdrossel
  mit realen Herstellerteilen und Digikey-Bestellnummern aufgesplittet
- NTC von 10R/3.5A (zu gering für 8A Lastpfad) auf Bourns BN-LG15Y2R5MYB
  (2.5R/8A) korrigiert
- cad/PoC KiCad-Projekt nach ECAD/IO_Board umbenannt (laufender Layout-Fortschritt)
- .gitignore um Backup-Ordner des neuen ECAD-Pfads ergänzt
Parts:
- added C1: C_X2_890334023023CS, aa_MyParts:C_Wurth_WCAP-FTXX-P10L13W7H13, F.Cu at (156.3, 128.8)
- added L1: L_CMC_7448258022, aa_MyParts:L_Wurth_WE-CMB-XL, F.Cu at (156.2, 114.6)
- added RV1: RVAR_B72210S0271K101, Varistor:RV_Disc_D12mm_W5.1mm_P7.5mm, F.Cu at (157.2, 120.0)
- added TH1: ICL_BN-LG15Y2R5MYB, Varistor:RV_Disc_D15.5mm_W8mm_P7.5mm, F.Cu at (172.0, 88.6)
- moved LED1 98.0 mm to (53.2, 82.1)
- moved PS1 98.0 mm to (59.3, 119.2)
- moved U1 98.0 mm to (13.7, 115.5)
- moved U2 98.0 mm to (80.2, 118.3)
- moved U3 98.0 mm to (54.5, 96.7)
- moved K2 98.0 mm to (67.0, 79.7)
- moved U4 98.0 mm to (70.7, 118.3)
- moved U5 98.0 mm to (46.0, 74.0)
- moved U6 98.0 mm to (46.8, 83.2)
- moved J2 93.5 mm to (231.3, 122.8)
- moved J1 74.2 mm to (173.1, 121.9)
- moved K1 70.3 mm to (196.2, 89.5), turned to 90 degrees
- moved F1 34.3 mm to (155.0, 88.9)
- renumbered J3 to F1
Connections:
- net Net-(J1-Pin_1) renamed /PIN_L
- net Net-(J1-Pin_3) renamed /PIN_N
- F1 pad 1: unconnected-(J3-Pad1) -> /PIN_CMC_L
- F1 pad 2: unconnected-(J3-Pad2) -> /PIN_FUSED_L
- J1 pad 5: Net-(J1-Pin_5) -> Earth
- J1 pad 6: Net-(J1-Pin_5) -> Earth
- J2 pad 5: Net-(J2-Pin_5) -> Earth
- J2 pad 6: Net-(J2-Pin_5) -> Earth
- K1 pad 2: unconnected-(K1-Pad2) -> Net-(J2-Pin_1)
- K1 pad 4: unconnected-(K1-Pad4) -> Net-(K1-Pad4)
- K1 pad 8: unconnected-(K1-Pad8) -> /PIN_CMC_N

Commit message: Optokoppler auf Vishay VO615A-X017T (verstärkte Isolierung) umgestellt, IO-Board Layout-Fortschritt
- PC817 durch Vishay VO615A-X017T ersetzt: VDE 0884-5 zertifizierte verstärkte
  Isolierung passend zur restlichen Schutzklasse-II-Auslegung (Relais, IRM-10-24),
  da der Optokoppler die einzige Isolationsbarriere der Lastmessung ist
- IO_Board KiCad-Projekt: Platzierungs-Fortschritt
Parts:
- removed K2: K_G5V-1-2_DC24, aa_MyParts:K_G5V-1-2_DC24
- removed LED1: LED_IN-PI20TATPRPGPB, aa_MyParts:LED_INPI20TATPRPGPB
- removed PS1: IC_R-78K5.0-2.0, aa_MyParts:IC_CONV_R-78K5.0-2.0
- removed U1: ESP32-S3-WROOM-1, RF_Module:ESP32-S3-WROOM-1
- removed U2: PN5321A3HN_C1xx, Package_DFN_QFN:HVQFN-40-1EP_6x6mm_P0.5mm_EP4.1x4.1mm
- added F2: 1A 250VAC, aa_MyParts:F_MRT_BEL, F.Cu at (83.6, 80.0)
- added R1: 20mR, Resistor_SMD:R_1206_3216Metric, F.Cu at (114.9, 94.3)
- added U7: VO615A-1, Package_DIP:DIP-4_W7.62mm, F.Cu at (102.9, 82.2)
- added U8: VO615A-1, Package_DIP:DIP-4_W7.62mm, F.Cu at (123.2, 79.4)
- moved U5 102.1 mm to (147.8, 67.1), turned to -90 degrees
- moved U4 74.9 mm to (134.1, 78.4), turned to 90 degrees
- moved J2 72.4 mm to (158.9, 124.0)
- moved L1 72.4 mm to (83.8, 115.7)
- moved F1 72.4 mm to (82.6, 90.1)
- moved C1 72.4 mm to (83.9, 130.0)
- moved J1 72.4 mm to (100.7, 123.1)
- moved K1 72.4 mm to (123.8, 90.7)
- moved RV1 72.4 mm to (84.8, 121.2)
- moved TH1 72.4 mm to (99.6, 89.7)
- moved U6 67.9 mm to (114.7, 84.0)
- moved U3 50.0 mm to (82.2, 55.0)
Connections:
- K1 pad 4: Net-(K1-Pad4) -> Net-(U6-I1-)
- TH1 pad 2: Net-(K1-Pad4) -> Net-(U6-V1+)
- U3 pad 1: unconnected-(U3-AC/N-Pad1) -> /PIN_CMC_N
- U3 pad 2: unconnected-(U3-AC/L-Pad2) -> Net-(U3-AC/L)
- U3 pad 3: unconnected-(U3--Vo-Pad3) -> Net-(U3--Vo)
- U4 pad 1: unconnected-(U4-GND-Pad1) -> Net-(U4-GND)
- U4 pad 2: unconnected-(U4-VO-Pad2) -> Net-(U4-VO)
- U4 pad 3: unconnected-(U4-VI-Pad3) -> Net-(U4-VI)
- U5 pad 2: unconnected-(U5--VIN-Pad2) -> Net-(U3--Vo)
- U5 pad 4: unconnected-(U5--VOUT-Pad4) -> Net-(U4-GND)
- U5 pad 6: unconnected-(U5-+VOUT-Pad6) -> Net-(U4-VI)
- U6 pad 12: unconnected-(U6-UART_TX-Pad12) -> Net-(U6-UART_TX)
- U6 pad 17: unconnected-(U6-I1--Pad17) -> Net-(U6-I1-)
- U6 pad 19: unconnected-(U6-V1+-Pad19) -> Net-(U6-V1+)
- U6 pad 25: unconnected-(U6-DVDD-Pad25) -> Net-(U4-VO)
- U6 pad 29: unconnected-(U6-DGND-Pad29) -> Net-(U4-GND)
- U6 pad 4: unconnected-(U6-UART_RX-Pad4) -> Net-(U6-UART_RX)
Other:
- board outline added: 100 x 100 mm
