File: hardware/projects/RFID_BOX/ECAD/IO_Board/IO_Board.kicad_pcb (KiCad board)
At the start: 2 copper layers, 90 x 98.5 mm, 72 parts, among them J300 J_WAGO_2604-1103, J301 J_WAGO_2604-1103, K300 T92S11D12-24, Q300 2N7002NXAKR, Q301 BSS84AK, Q302 2N7002NXAKR, U300 ISOW7721DFMR, U301 IRM-10-24, U302 MCP39F511A-E/MQ, U306 R-78K5.0-2.0, U307 AP2114H-3.3TRG1

Commit message: IO_Board: Review-Antworten umgesetzt, Sicherungskonzept überarbeitet
Schaltplan:
- Entladekette R305-R310-R321, drei 330k in Reihe parallel zu RV300/C300:
  990 kOhm, C300 unter 60 V in 0,17 s, je Widerstand 77 V effektiv (F1)
- Tiefpass an ISO_EN: R322 1k in Reihe, C329 10nF gegen GND1 (F9)
- FB300 im Abgriff des HV-Teilers entfernt, gegen 1 MOhm wirkungslos (F8)
- F301 von Schurter 0034.3127 auf Bel 5HT 10-R: Keramik sandgefuellt,
  Ausschaltvermoegen 1500 A statt 100 A (F10)
- R323 Sicherungswiderstand 10 Ohm vor F302, begrenzt den Fehlerstrom
  auf 25 A und damit unter die 35 A der MRT (F11)
- R319/R320 als 0R-Bruecken in den UART-Leitungen zu U302

README:
- Abstandsmatrix als Mastertabelle mit L, N, ISO-Insel, SELV, PE und FELD;
  loest die alte Fassung mit NETZ gleicher Pol / Gegenpol ab
- Netzklassen L und N dokumentiert, zugeordnet ueber /PIN_L* und /PIN_N*,
  orthogonal zu den Breitenklassen 230V_ext und 230V_int
- ISO-Insel liegt ueber NT300 auf N-Potential: 0,5 mm gegen N, 3,0 mm gegen L
- Verweis auf den Regelsatz IO_Board.kicad_dru und die U300-Ausnahme
- Bauteiltabellen: Entladekette, R322, R323, F301, Ferritzeile auf FB301/FB302
- FMEA: vier Zeilen fuer F301, F302, Entladekette und Q301 im Linearbetrieb,
  Relaistreiber-Zeile um die Steckerbelegung auf J302 ergaenzt

Datenblaetter: Bel 5HT, Vishay PR01

Co-Authored-By: Claude Opus 5 <noreply@anthropic.com>
Parts:
- removed FB300: 600R@100MHz, Inductor_SMD:L_0805_2012Metric
- added C329: 10nF, Capacitor_SMD:C_0603_1608Metric, F.Cu at (176.4, 122.7)
- added R305: 330k, Resistor_SMD:R_0805_2012Metric, F.Cu at (172.2, 122.9)
- added R310: 330k, Resistor_SMD:R_0805_2012Metric, F.Cu at (172.2, 125.8)
- added R321: 330k, Resistor_SMD:R_0805_2012Metric, F.Cu at (175.9, 130.5)
- added R322: 1k, Resistor_SMD:R_0603_1608Metric, F.Cu at (176.4, 125.2)
- added R323: 10R, Resistor_THT:R_Axial_DIN0207_L6.3mm_D2.5mm_P15.24mm_Horizontal, F.Cu at (78.4, 103.1)
- moved F302 5.76 mm to (82.2, 91.2)
- moved C309 2.32 mm to (94.0, 83.0)
- moved C310 2.22 mm to (88.5, 83.1)
- moved L300 0.28 mm to (91.7, 101.2)
Connections:
- net ISO_EN renamed Net-(U300-EN)
- F302 pad 1: /PIN_L -> Net-(F302-Pad1)
- R303 pad 1: /PIN_L_SENSE -> /PIN_L_FUSED

Commit message: IO_Board: Shunt R300 auf pulsfesten CSI2H-2512K-2L00G, Schema V1.2
R300 von CRF2010-FZ-R002ELF auf Bourns CSI2H-2512K-2L00G: 2mOhm +-2%,
+-75ppm/K, 5W @70C, 2512. Sense-Abgriffe liegen wieder auf /PIN_N und
/PIN_N_SHUNT, ERC ohne duplicate_pins, PCB nachgezogen.

README: Shunt-Zeile und Engstellen-Notiz zum Lastpfad aktualisiert,
BOM neu exportiert, Datenblatt abgelegt.

Co-Authored-By: Claude Opus 5 <noreply@anthropic.com>
Parts:
- R300: footprint Resistor_SMD:R_2010_5025Metric -> aa_MyParts:R_2512_CSI2H-2512K-2L00G
- moved R300 4.07 mm to (99.8, 116.2)
Connections:
- R300 pad 1: /PIN_N -> /PIN_N_SHUNT
- R300 pad 2: /PIN_N_SHUNT -> /PIN_N
Changed lines of the file:
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@@
 		)
 	)
-	(footprint "Resistor_SMD:R_2010_5025Metric"
-		(layer "F.Cu")
-		(at 97.917 112.573)
-		(descr "Resistor SMD 2010 (5025 Metric), square (rectangular) end terminal, IPC-7351 nominal, (Body size source: IPC-SM-782 page 72, https://www.pcb-3d.com/wordpress/wp-content/uploads/ipc-sm-782a_amendment_1_and_2.pdf)")
-		(tags "resistor")
-		(property "Reference" "R300"
-			(at 0 -2.28 0)
-			(layer "F.SilkS")
-			(effects
-				(font
-					(size 1 1)
-					(thickness 0.15)
-				)
-			)
-		)
-		(property "Value" "2mR"
-			(at 0 2.28 0)
-			(layer "F.Fab")
-			(effects
-				(font
-					(size 1 1)
-					(thickness 0.15)
-				)
-			)
-		)
-		(property "Datasheet" "https://www.mouser.com/catalog/specsheets/Bourns_6-27-2025_CRF_Datasheet.pdf"
-			(at 0 0 0)
-			(layer "F.Fab")
-			(hide yes)
-			(effects
-				(font
-					(size 1.27 1.27)
-				)
-			)
-		)
-		(property "Description" "Resistor"
-			(at 0 0 0)
-			(layer "F.Fab")
-			(hide yes)
-			(effects
-				(font
-					(size 1.27 1.27)
-				)
-			)
-		)
-		(property "Manufacturer" "Bourns Inc."
-			(at 0 0 0)
-			(unlocked yes)
-			(layer "F.Fab")
-			(hide yes)
-			(effects
-				(font
-					(size 1 1)
-					(thickness 0.15)
-				)
-			)
-		)
-		(property "Manufacturer Part Number" "CRF2010-FZ-R002ELF"
-			(at 0 0 0)
-			(unlocked yes)
-			(layer "F.Fab")
-			(hide yes)
-			(effects
-				(font
-					(size 1 1)
-					(thickness 0.15)
-				)
-			)
-		)
-		(property "Distributor 1" "Mouser"
-			(at 0 0 0)
-			(unlocked yes)
-			(layer "F.Fab")
-			(hide yes)
-			(effects
-				(font
-					(size 1 1)
-					(thickness 0.15)
-				)
-			)
-		)
-		(property "Distributor 1 Order Number" "652-CRF2010FZR002ELF"
-			(at 0 0 0)
-			(unlocked yes)
-			(layer "F.Fab")
-			(hide yes)
-			(effects
-				(font
-					(size 1 1)
-					(thickness 0.15)
-				)
-			)
-		)
-		(property "Distributor 2" "Digi-Key"
-			(at 0 0 0)
-			(unlocked yes)
-			(layer "F.Fab")
-			(hide yes)
-			(effects
-				(font
-					(size 1 1)
-					(thickness 0.15)
-				)
-			)
-		)
-		(property "Distributor 2 Order Number" "118-CRF2010-FZ-R002ELFCT-ND"
-			(at 0 0 0)
-			(unlocked yes)
-			(layer "F.Fab")
-			(hide yes)
-			(effects
-				(font
-					(size 1 1)
-					(thickness 0.15)
-				)
-			)
-		)
-		(property ki_fp_filters "R_*")
-		(sheetname "/")
-		(sheetfile "IO_Board.kicad_sch")
-		(units
-			(unit
-				(name "A")
-				(pins "1" "2")
-			)
-		)
-		(attr smd)
-		(duplicate_pad_numbers_are_jumpers no)
-		(fp_line
-			(start -1.527064 -1.36)
-			(end 1.527064 -1.36)
-			(stroke
-				(width 0.12)
-				(type solid)
-			)
-			(layer "F.SilkS")
-		)
-		(fp_line
-			(start -1.527064 1.36)
-			(end 1.527064 1.36)
-			(stroke
-				(width 0.12)
-				(type solid)
-			)
-			(layer "F.SilkS")
-		)
-		(fp_rect
-			(start -3.18 -1.58)
-			(end 3.18 1.58)
-			(stroke
-				(width 0.05)
-				(type solid)
-			)
-			(fill no)
-			(layer "F.CrtYd")
-		)
-		(fp_rect
-			(start -2.5 -1.25)
-			(end 2.5 1.25)
-			(stroke
-				(width 0.1)
-				(type solid)
-			)
-			(fill no)
-			(layer "F.Fab")
-		)
-		(fp_text user "${REFERENCE}"
-			(at 0 0 0)
-			(layer "F.Fab")
-			(effects
-				(font
-					(size 1 1)
-					(thickness 0.15)
-				)
-			)
-		)
-		(pad "1" smd roundrect
-			(at -2.3125 0)
-			(size 1.225 2.65)
-			(layers "F.Cu" "F.Mask" "F.Paste")
-			(roundrect_rratio 0.204082)
-			(net "/PIN_N")
-			(pintype "passive")
-		)
-		(pad "2" smd roundrect
-			(at 2.3125 0)
-			(size 1.225 2.65)
-			(layers "F.Cu" "F.Mask" "F.Paste")
-			(roundrect_rratio 0.204082)
-			(net "/PIN_N_SHUNT")
-			(pintype "passive")
-		)
-		(embedded_fonts no)
-		(model "${KICAD10_3DMODEL_DIR}/Resistor_SMD.3dshapes/R_2010_5025Metric.step"
-			(offset
-				(xyz 0 0 0)
-			)
-			(scale
-				(xyz 1 1 1)
-			)
-			(rotate
-				(xyz 0 0 0)
-			)
-		)
-	)
 	(footprint "Capacitor_SMD:C_0603_1608Metric"
 		(layer "F.Cu")
@@
 			)
 		)
+	)
+	(footprint "aa_MyParts:R_2512_CSI2H-2512K-2L00G"
+		(layer "F.Cu")
+		(at 99.755 116.2)
+		(descr "Resistor SMD 2512 (6332 Metric), square (rectangular) end terminal, IPC-7351 nominal, (Body size source: IPC-SM-782 page 72, https://www.pcb-3d.com/wordpress/wp-content/uploads/ipc-sm-782a_amendment_1_and_2.pdf)")
+		(tags "resistor")
+		(property "Reference" "R300"
+			(at 0 -2.63 0)
+			(layer "F.SilkS")
+			(effects
+				(font
+					(size 1 1)
+					(thickness 0.15)
+				)
+			)
+		)
+		(property "Value" "2mR"
+			(at 0 2.63 0)
+			(layer "F.Fab")
+			(effects
+				(font
+					(size 1 1)
+					(thickness 0.15)
+				)
+			)
+		)
+		(property "Datasheet" "https://www.mouser.com/catalog/specsheets/Bourns_11152023_CSI2H-2512_Datasheet.pdf?_gl=1*f4tsx1*_gcl_au*MTQ0ODQ4Nzc3OS4xNzg1MDYwNjMzLjEzNDA3NTc3NzMuMTc5MjgzMTQ2Ni4xNzkyODMyNTQ4LjEzOTIzMTc2NjQuMTc5MjgzMTQ2Ni4xNzkyODMyNTQ4*_ga*NTkzNzgzMTMxLjE3ODUwNjA2MzM.*_ga_15W4STQT4T*czE3OTI4MzE0MjkkbzIyJGcxJHQxNzkyODMyNzA3JGo2MCRsMCRoMA.."
+			(at 0 0 0)
+			(layer "F.Fab")
+			(hide yes)
+			(effects
+				(font
+					(size 1.27 1.27)
+				)
+			)
+		)
+		(property "Description" "Resistor"
+			(at 0 0 0)
+			(layer "F.Fab")
+			(hide yes)
+			(effects
+				(font
+					(size 1.27 1.27)
+				)
+			)
+		)
+		(property "Manufacturer" "Bourns Inc."
+			(at 0 0 0)
+			(unlocked yes)
+			(layer "F.Fab")
+			(hide yes)
+			(effects
+				(font
+					(size 1 1)
+					(thickness 0.15)
+				)
+			)
+		)
+		(property "Manufacturer Part Number" "CSI2H-2512K-2L00G"
+			(at 0 0 0)
+			(unlocked yes)
+			(layer "F.Fab")
+			(hide yes)
+			(effects
+				(font
+					(size 1 1)
+					(thickness 0.15)
+				)
+			)
+		)
+		(property "Distributor 1" "Mouser"
+			(at 0 0 0)
+			(unlocked yes)
+			(layer "F.Fab")
+			(hide yes)
+			(effects
+				(font
+					(size 1 1)
+					(thickness 0.15)
+				)
+			)
+		)
+		(property "Distributor 1 Order Number" "652-CSI2H-2512K2L00G"
+			(at 0 0 0)
+			(unlocked yes)
+			(layer "F.Fab")
+			(hide yes)
+			(effects
+				(font
+					(size 1 1)
+					(thickness 0.15)
+				)
+			)
+		)
+		(property "Distributor 2" "Digi-Key"
+			(at 0 0 0)
+			(unlocked yes)
+			(layer "F.Fab")
+			(hide yes)
+			(effects
+				(font
+					(size 1 1)
+					(thickness 0.15)
+				)
+			)
+		)
+		(property "Distributor 2 Order Number" "118-CSI2H-2512K-2L00GETR-ND"
+			(at 0 0 0)
+			(unlocked yes)
+			(layer "F.Fab")
+			(hide yes)
+			(effects
+				(font
+					(size 1 1)
+					(thickness 0.15)
+				)
+			)
+		)
+		(property ki_fp_filters "R_*")
+		(sheetname "/")
+		(sheetfile "IO_Board.kicad_sch")
+		(units
+			(unit
+				(name "A")
+				(pins "1" "2")
+			)
+		)
+		(attr smd)
+		(duplicate_pad_numbers_are_jumpers no)
+		(fp_line
+			(start -2.177064 -1.71)
+			(end 2.177064 -1.71)
+			(stroke
+				(width 0.12)
+				(type solid)
+			)
+			(layer "F.SilkS")
+		)
+		(fp_line
+			(start -2.177064 1.71)
+			(end 2.177064 1.71)
+			(stroke
+				(width 0.12)
+				(type solid)
+			)
+			(layer "F.SilkS")
+		)
+		(fp_rect
+			(start -3.83 -1.93)
+			(end 3.83 1.93)
+			(stroke
+				(width 0.05)
+				(type solid)
+			)
+			(fill no)
+			(layer "F.CrtYd")
+		)
+		(fp_rect
+			(start -3.15 -1.6)
+			(end 3.15 1.6)
+			(stroke
+				(width 0.1)
+				(type solid)
+			)
+			(fill no)
+			(layer "F.Fab")
+		)
+		(fp_text user "${REFERENCE}"
+			(at 0 0 0)
+			(layer "F.Fab")
+			(effects
+				(font
+					(size 1 1)
+					(thickness 0.15)
+				)
+			)
+		)
+		(pad "1" smd roundrect
+			(at -2.6 0)
+			(size 1.8 3.4)
+			(layers "F.Cu" "F.Mask" "F.Paste")
+			(roundrect_rratio 0)
+			(chamfer_ratio 0.2)
+			(chamfer top_right bottom_right)
+			(net "/PIN_N_SHUNT")
+			(pintype "passive")
+		)
+		(pad "2" smd roundrect
+			(at 2.6 0)
+			(size 1.8 3.4)
+			(layers "F.Cu" "F.Mask" "F.Paste")
+			(roundrect_rratio 0)
+			(chamfer_ratio 0.2)
+			(chamfer top_left bottom_left)
+			(net "/PIN_N")
+			(pintype "passive")
+		)
+		(embedded_fonts no)
+		(model "/Users/marius/Github/MyCSLib/3D_Models/Res/R_CSI2H-2512.stp"
+			(offset
+				(xyz -3.2 -1.5 0)
+			)
+			(scale
+				(xyz 1 1 1)
+			)
+			(rotate
+				(xyz -90 -0 -0)
+			)
+		)
