File: hardware/projects/RFID_BOX/ECAD/IO_Board/IO_Board.kicad_sch (KiCad schematic)
At the start: 39 parts, among them J300 J_WAGO_2604-1103, J301 J_WAGO_2604-1103, K300 T92S11D12-24, U300 IC_ISOW7721DFMR, U301 IRM-10-24, U303 MCP39F511A-E/MQ, U306 R-78K5.0-2.0

Commit message: update from lib
Parts:
- C300: Distributor 1 (none) -> Mouser; Distributor 2 (none) -> Digi-Key; Distributor 2 Order Number (none) -> *732-5733-ND; Manufacturer (none) -> *Wurth Elektronik; Manufacturer Part Number (none) -> *890334023023CS
- C302: Distributor 1 (none) -> Mouser; Distributor 2 (none) -> Digi-Key; Distributor 2 Order Number (none) -> *732-8664-1-ND; Manufacturer (none) -> *Wurth Elektronik; Manufacturer Part Number (none) -> 860010673012
- C309, C310: Distributor 1 (none) -> Mouser; Distributor 2 (none) -> Digi-Key; Distributor 2 Order Number (none) -> *VY2472M49Y5US63L7-ND; Manufacturer (none) -> *Vishay BC Components; Manufacturer Part Number (none) -> *VY2472M49Y5US63L7
- F300: Distributor 1 (none) -> Mouser; Distributor 2 (none) -> Digi-Key; Distributor 2 Order Number (none) -> *732-11383-ND; Manufacturer Part Number (none) -> 696309001002
- F302: Distributor 1 (none) -> Mouser; Distributor 2 (none) -> Digi-Key; Distributor 2 Order Number (none) -> *5923-MRT500-BULK-ND; Manufacturer (none) -> *Bel Fuse; Manufacturer Part Number (none) -> *MRT 500-BULK
- FB300, FB301, FB302: Distributor 1 (none) -> Mouser; Distributor 2 (none) -> Digi-Key; Distributor 2 Order Number (none) -> *MH2029-601YCT-ND; Manufacturer (none) -> *Bourns; Manufacturer Part Number (none) -> *MH2029-601Y
- FB303, FB304, FB305, FB306, FB307: Current (none) -> 1A; DCR (none) -> 200mR; Distributor 1 (none) -> Mouser; Distributor 2 (none) -> Digi-Key; Distributor 2 Order Number (none) -> *MH2029-601YCT-ND; Manufacturer (none) -> *Bourns; Manufacturer Part Number (none) -> *MH2029-601Y
- J300, J301: Distributor 1 (none) -> Mouser; Distributor 2 (none) -> Digi-Key; Distributor 2 Order Number (none) -> *2946-2604-1103-ND; Manufacturer (none) -> *WAGO; Manufacturer Part Number (none) -> *2604-1103
- K300: Distributor 1 (none) -> Mouser; Distributor 2 (none) -> Digi-Key; Distributor 2 Order Number (none) -> *PB352-ND; Manufacturer (none) -> *TE Connectivity Potter & Brumfield; Manufacturer Part Number (none) -> *T92S11D12-24
- L300: Distributor 1 (none) -> Mouser; Distributor 2 (none) -> Digi-Key; Distributor 2 Order Number (none) -> *817-2084-ND; Manufacturer Part Number (none) -> RN102-1-02-3M0
- RV300: Distributor 1 (none) -> Mouser; Distributor 2 (none) -> Digi-Key; Distributor 2 Order Number (none) -> *495-3786-ND; Manufacturer (none) -> *TDK (EPCOS); Manufacturer Part Number (none) -> *B72210S0271K101
- U300: Distributor 1 (none) -> Mouser; Distributor 2 (none) -> Digi-Key; Distributor 2 Order Number (none) -> *296-ISOW7721DFMRCT-ND; Manufacturer (none) -> *Texas Instruments; Manufacturer Part Number (none) -> *ISOW7721DFMR
- U301: Distributor 1 (none) -> Mouser; Distributor 2 (none) -> Digi-Key; Distributor 2 Order Number (none) -> *1866-3030-ND; Manufacturer (none) -> *MEAN WELL; Manufacturer Part Number (none) -> *IRM-10-24
- U303: Distributor 1 (none) -> Mouser; Distributor 2 (none) -> Digi-Key; Distributor 2 Order Number (none) -> *MCP39F511A-E/MQ-ND; Manufacturer (none) -> *Microchip Technology; Manufacturer Part Number (none) -> *MCP39F511A-E/MQ
- U306: Distributor 1 (none) -> Mouser; Distributor 2 (none) -> Digi-Key; Distributor 2 Order Number (none) -> *945-R-78K5.0-2.0-ND; Manufacturer (none) -> Recom Power; Manufacturer Part Number (none) -> R-78K5.0-2.0
