File: hardware/projects/RFID_BOX/ECAD/IO_Board/IO_Board.kicad_sch (KiCad schematic)
At the start: 39 parts, among them J300 J_WAGO_2604-1103, J301 J_WAGO_2604-1103, K300 T92S11D12-24, U300 IC_ISOW7721DFMR, U301 IRM-10-24, U303 MCP39F511A-E/MQ, U306 R-78K5.0-2.0

Commit message: Relaistreiber bestueckt, README gestrafft
Treiber des Lastrelais vollstaendig ausgelegt: Low-Side-NMOS Q300 und
High-Side-PMOS Q301 in Reihe in der Spule, dazu Q302 als Pegelwandler
fuer den symmetrischen 47k/47k-Gate-Teiler von Q301. Die Symmetrie ist
zwingend, unsymmetrisch laege Vgs ueber dem Gate-Limit von +/-20V.

Bauteile: 2N7002NXAKR (Q300, Q302), BSS84AK (Q301), BAS16LT1G (D305).
D305 bleibt im SOT-23 statt SOD-323 — verdrehsicher und in der
Groessenklasse der 0603-Passiven. BOM-Summe 90,11 -> 90,00 EUR.

README: Kapitel "Versorgung und Isolation der Messinsel" und der
Relaistreiber-Abschnitt entfallen; die 4mm-Kupfersperrzone um VISOOUT
und die Ferrit-Trennung GND_ISO2/GND_ISO sind nach "Domaenen und
Abstaende" gewandert. Acht erledigte oder nicht mehr relevante
TODO-Eintraege geloescht.

Datenblaetter fuer die neuen Bauteile ergaenzt.

Co-Authored-By: Claude Opus 5 <noreply@anthropic.com>
Parts:
- removed U303: MCP39F511A-E/MQ, aa_MyParts:IC_QFN28_MQ_MCH, symbol aa_MyParts:IC_MCP39F511A-E_MQ
- added C318, C319, C320, C321: 33nF 50V, Capacitor_SMD:C_0603_1608Metric, symbol Device:C
- added C322: 1uF 10V, Capacitor_SMD:C_0603_1608Metric, symbol Device:C
- added C323, C324, C327: 100nF 25V, Capacitor_SMD:C_0603_1608Metric, symbol Device:C
- added C325: 10uF, Capacitor_SMD:C_0603_1608Metric, symbol Device:C
- added C326: 10uF 10V, Capacitor_SMD:C_0805_2012Metric, symbol Device:C
- added C328: 10uF 10V 0805, Capacitor_SMD:C_0805_2012Metric, symbol Device:C
- added D300: D_BAS16LT1G, Package_TO_SOT_SMD:SOT-23, symbol aa_MyParts:D_BAS16LT1G
- added unit 1 of K300
- added NT300: NetTie, NetTie:NetTie-2_SMD_Pad0.5mm, symbol Device:NetTie_2
- added PS300: AP2114H-3.3TRG1, Package_TO_SOT_SMD:SOT-223-3_TabPin2, symbol aa_MyParts:IC_AP2114H-3.3TRG1
- added Q300, Q302: 2N7002NXAKR, Package_TO_SOT_SMD:SOT-23, symbol aa_MyParts:Q_NMOS_2N7002NXAKR
- added Q301: BSS84AK, Package_TO_SOT_SMD:SOT-23, symbol aa_MyParts:Q_PMOS_BSS84AK
- added R301, R302, R306, R312, R315: 1k, Resistor_SMD:R_0603_1608Metric, symbol Device:R
- added R303, R304: 499k, Resistor_SMD:R_2010_5025Metric, symbol Device:R
- added R307: 10R, Resistor_SMD:R_0603_1608Metric, symbol Device:R
- added R308, R309, R311: 2k, Resistor_SMD:R_0603_1608Metric, symbol Device:R
- added R310: 2R49, Resistor_SMD:R_0603_1608Metric, symbol Device:R
- added R313, R314, R316, R317: 47k, Resistor_SMD:R_0603_1608Metric, symbol Device:R
- added U302: MCP39F511A-E/MQ, aa_MyParts:IC_QFN28_MQ_MCH, symbol aa_MyParts:IC_MCP39F511A-E_MQ
- C301, C304, C305, C306, C307, C308, C311, C312, C313, C314, C315, C316, C317: footprint (none) -> Capacitor_SMD:C_0603_1608Metric
- C303: footprint (none) -> Capacitor_SMD:C_0805_2012Metric
- R300: value 2mR PA1206FRM670R002L -> 2mR CRF2010-FZ-R002ELF; footprint Resistor_SMD:R_1206_3216Metric -> Resistor_SMD:R_2010_5025Metric
- U300: value IC_ISOW7721DFMR -> ISOW7721DFMR
Connections:
- net +24V: now also Q301.2 (S), R313.2
- net +3V3: now also FB306.2, C325.1, PS300.2 (+VOUT)
- net +3V3_ISO: now also FB303.1, U300.17 (EN_IO2), C324.1, R307.1, R311.1, U302.10 (nRESET), U302.25 (DVDD); no longer FB303.2
- net +5V: now also C328.1, PS300.3 (+VIN)
- net GND: now also C325.2, C328.2, PS300.1 (GND), Q300.2 (S), Q302.2 (S), R316.1, R317.1; no longer U300.7 (LF)
- net GND_ISO: now also FB304.1, C318.2, C319.1, C320.2, C321.2, C322.2, C323.2, C324.2, C326.2, C327.2, NT300.1, R306.1, R308.1, R309.1, U302.21 (AGND), U302.24 (DGND), U302.27 (DGND), U302.29 (DGND); no longer FB304.2
- net PIN_N: now also NT300.2
- net UART_MCP2MCU_ISO: now also U302.12 (UART_TX)
- net UART_MCU2MCP_ISO: now also U302.4 (UART_RX)
- net V_ISO_OUT: now reaches C315.1, C316.1, C317.1, U300.12 (V_{ISOOUT})
- net V_ISO_OUT: now also FB303.2; no longer FB303.1
- net VIO: now reaches C304.1, C305.1, C306.1, FB306.1, U300.1 (V_{IO})
- net VIO: no longer U300.5 (EN)
- net VDD: now reaches U300.4 (EN_IO1)
- net VDD: now also C307.1, C308.1, C311.1, FB307.1, U300.5 (EN), U300.9 (V_{DD})
- net at FB302.1: now also R302.1, R310.1
- net at FB301.1: now also R301.1, R310.2
- net at FB300.1: now also R303.1
- net GND2 renamed GND1
- net GND1: now also U300.7 (LF)
- net GND_ISO2 renamed GND2_ISO
- net GND2_ISO: now also FB304.2; no longer FB304.1
- new net: D300.1 (A), K300.0, Q300.3 (D)
- new net: D300.3 (K), K300.1, Q301.3 (D)
- new net: C321.1, R306.2, U302.19 (V1+)
- new net: Q300.1 (G), R312.1, R316.2
- new net: R303.2, R304.1
- new net: Q302.1 (G), R315.1, R317.2
- new net: Q302.3 (D), R314.1
- new net: C326.1, C327.1, U302.23 (REFIN+/OUT)
- new net: C322.1, C323.1, R307.2, U302.11 (AVDD)
- new net: U302.13 (COMMONB), U302.5 (COMMONA)
- new net: C318.1, R301.2, U302.16 (I1+)
- new net: C319.2, R302.2, U302.17 (I1-)
- new net: C320.1, R304.2, R308.2, R309.2, U302.18 (V1-)
- new net: R311.2, U302.26 (nMCLR)
- new net: Q301.1 (G), R313.1, R314.2
- no-connect marks 5 -> 13
Other:
- note added: "Digital isolator with integrated DC/DC In: 3.3VDC (VDD = VIO) Out: 3.3VDC, 60mA, 24mVpp ripple Ch: 1 forward + 1 reverse, 100Mbps Fail-safe output HIGH (no F suffix) Eff: 46% @ max load Iso: Reinforced per VDE 0884-17, 5kVrms/60s 1000Vrms working, >8mm creepage/clearance CTI >600V, material group I Protection: Soft-start, UVLO, OVP Overload, short-circuit, thermal shutdown"
- note added: "Relay coil, K300 (TE T92S11D12-24) Coil: 24VDC, 350R ±10%, 1.7W Current: 69mA nom, 76mA @ -10% R Thresholds: Operate 18V, Release 2.4V Iso: 4kV coil-to-contact, 8mm air / 9.5mm surface Insulation: Class F, 155C max coil temp"
- moved on the sheet: C300, C301, C302, C303, C304, C305, C306, C307, C308, C309, C310, C311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
