File: hardware/projects/RFID_BOX/ECAD/IO_Board/IO_Board.kicad_sch (KiCad schematic)
At the start: 72 parts, among them J300 J_WAGO_2604-1103, J301 J_WAGO_2604-1103, K300 T92S11D12-24, Q300 2N7002NXAKR, Q301 BSS84AK, Q302 2N7002NXAKR, U300 ISOW7721DFMR, U301 IRM-10-24, U302 MCP39F511A-E/MQ, U306 R-78K5.0-2.0

Commit message: fix some parts
Parts:
- removed K300: T92S11D12-24, aa_MyParts:K_T92S11D12-24, symbol aa_MyParts:T92S11D12-24
- added J302: Conn_01x10_Pin, symbol Connector:Conn_01x10_Pin
- added K300: T92S11D12-24, aa_MyParts:K_T92S11D12-24, symbol aa_MyParts:K_T92S11D12-24
- C300: Distributor 1 Order Number (none) -> 710-890334023023CS; Distributor 2 Order Number *732-5733-ND -> 732-5733-ND; Manufacturer *Wurth Elektronik -> Wurth Elektronik; Manufacturer Part Number *890334023023CS -> 890334023023CS
- C302: Distributor 1 Order Number (none) -> 710-860010673012; Distributor 2 Order Number *732-8664-1-ND -> 732-8664-1-ND; Manufacturer *Wurth Elektronik -> Wurth Elektronik
- C309, C310: Distributor 1 Order Number (none) -> 72-VY2472M49Y5US63L7; Distributor 2 Order Number *VY2472M49Y5US63L7-ND -> VY2472M49Y5US63L7-ND; Manufacturer *Vishay BC Components -> Vishay BC Components; Manufacturer Part Number *VY2472M49Y5US63L7 -> VY2472M49Y5US63L7
- D300: Distributor 1 (none) -> Mouser; Distributor 1 Order Number (none) -> 863-BAS16LT1G; Distributor 2 (none) -> Digi-Key; Distributor 2 Order Number (none) -> BAS16LT1GOSCT-ND; Manufacturer (none) -> onsemi; Manufacturer Part Number (none) -> BAS16LT1G
- F300: Distributor 1 Order Number (none) -> 710-696309001002; Distributor 2 Order Number *732-11383-ND -> 732-11383-ND
- F302: Distributor 1 Order Number (none) -> 530-MRT500BULKSHORT; Distributor 2 Order Number *5923-MRT500-BULK-ND -> 5923-MRT500-BULK-ND; Manufacturer *Bel Fuse -> Bel Fuse; Manufacturer Part Number *MRT 500-BULK -> MRT 500-BULK
- FB300, FB301, FB302, FB303, FB304, FB305, FB306, FB307: Distributor 1 Order Number (none) -> 652-MH2029-601Y; Distributor 2 Order Number *MH2029-601YCT-ND -> MH2029-601YCT-ND; Manufacturer *Bourns -> Bourns; Manufacturer Part Number *MH2029-601Y -> MH2029-601Y
- J300, J301: Distributor 1 Order Number (none) -> n/A; Distributor 2 Order Number *2946-2604-1103-ND -> 2946-2604-1103-ND; Manufacturer *WAGO -> WAGO; Manufacturer Part Number *2604-1103 -> 2604-1103
- L300: Distributor 1 Order Number (none) -> 631-RN102-1-02-3M0; Distributor 2 Order Number *817-2084-ND -> 817-2084-ND
- PS300: Distributor 1 Order Number (none) -> 621-AP2114H-3.3TRG1
- Q300, Q302: Distributor 1 Order Number (none) -> 771-2N7002NXAKR; Distributor 2 Order Number (none) -> 1727-8643-1-ND; Manufacturer (none) -> Nexperia USA Inc.; Manufacturer Part Number (none) -> 2N7002NXAKR
- Q301: Distributor 1 (none) -> Mouser; Distributor 1 Order Number (none) -> 771-BSS84AK215; Distributor 2 (none) -> Digi-Key; Distributor 2 Order Number (none) -> 1727-1144-1-ND; Manufacturer (none) -> Nexperia USA Inc.; Manufacturer Part Number (none) -> BSS84AK,215
- RV300: Distributor 1 Order Number (none) -> 871-B72210S271K101; Distributor 2 Order Number *495-3786-ND -> 495-3786-ND; Manufacturer *TDK (EPCOS) -> TDK (EPCOS); Manufacturer Part Number *B72210S0271K101 -> B72210S0271K101
- U300: Distributor 1 Order Number (none) -> 595-ISOW7721DFMR; Distributor 2 Order Number *296-ISOW7721DFMRCT-ND -> 296-ISOW7721DFMRCT-ND; Manufacturer *Texas Instruments -> Texas Instruments; Manufacturer Part Number *ISOW7721DFMR -> ISOW7721DFMR
- U301: Distributor 1 Order Number (none) -> 709-IRM10-24; Distributor 2 Order Number *1866-3030-ND -> 1866-3030-ND; Manufacturer *MEAN WELL -> MEAN WELL; Manufacturer Part Number *IRM-10-24 -> IRM-10-24
- U302: Distributor 1 Order Number (none) -> 579-MCP39F511AE/MQ; Distributor 2 Order Number *MCP39F511A-E/MQ-ND -> MCP39F511A-E/MQ-ND; Manufacturer *Microchip Technology -> Microchip Technology; Manufacturer Part Number *MCP39F511A-E/MQ -> MCP39F511A-E/MQ
- U306: Distributor 1 Order Number (none) -> 919-R-78K5.0-2.0; Distributor 2 Order Number *945-R-78K5.0-2.0-ND -> 945-R-78K5.0-2.0-ND
Connections:
- net +24V: now also J302.1 (Pin_1)
- net +3V3: now also J302.5 (Pin_5)
- net +5V: now also J302.3 (Pin_3)
- net GND: now also J302.10 (Pin_10), J302.2 (Pin_2), J302.4 (Pin_4)
- net PIN_FUSED_L: now also K300.4
- net UART_MCP2MCU: now also J302.7 (Pin_7)
- net UART_MCU2MCP: now also J302.6 (Pin_6)
- net at D300.1 (A), Q300.3 (D): now also K300.0
- net at D300.3 (K), Q301.3 (D): now also K300.1
- net at FB302.2, R300.2: now also K300.8
- net at J301.1 (Pin_1), J301.2 (Pin_2): now also K300.2
- net at J301.3 (Pin_3), J301.4 (Pin_4): now also K300.6
- net relay_en_LS: now reaches R312.2
- net relay_en_LS: now also J302.9 (Pin_9)
- net relay_en_HS: now reaches R315.2
- net relay_en_HS: now also J302.8 (Pin_8)
- no-connect marks 13 -> 15
Other:
- note removed: "Common Mode Choke"
- moved on the sheet: L300, R303
