File: hardware/projects/RFID_BOX/ECAD/IO_Board/IO_Board.kicad_sch (KiCad schematic)
At the start: 73 parts, among them J300 J_WAGO_2604-1103, J301 J_WAGO_2604-1103, J302 Conn_01x10_Pin, K300 T92S11D12-24, Q300 2N7002NXAKR, Q301 BSS84AK, Q302 2N7002NXAKR, U300 ISOW7721DFMR, U301 IRM-10-24, U302 MCP39F511A-E/MQ, U306 R-78K5.0-2.0

Commit message: IO_Board 230V reviewfertig, README nachgezogen
Schaltplan:
- PE als ein Netz (PIN_PE) inkl. Y-Mittelabgriff C309/C310
- FB305 entfernt, GND1/GNDIO/LF von U300 zusammen auf GND (Datenblatt)
- Ferrite FB303/304/306/307 auf BLM15EX331SN1D 330R 0402
- R310 entfernt, Stromkanal als reine Kelvin-Messung
- ISO_EN von U300 Pin 5 auf J302.4, Pull-up R318 47k nach VDD
- OSCI/OSCO von U302 NC, interner 4-MHz-Oszillator
- PIN_L_SWITCHED / PIN_N_SWITCHED benannt, PS300 zu U307 umbenannt
- R300 und F301 mit Hersteller, MPN, Datenblatt und Bestellnummern
- aa_MyParts: AGND/DGND von U302 als Power Input
- ERC 0 Fehler (power_pin_not_driven und pin_not_driven auf ignore)

README:
- RC-Snubber gestrichen: der Node ist Lastschalter
- Netznamen an den Schaltplan angeglichen
- Erledigte TODOs zu GND1/GNDIO und den VIO/VDD-Ferriten entfernt
- Gain 16/1, ISO_EN-Reset, 3V3-Zeile in der Leiterbahntabelle
- BOM: R318, FB300-FB302, Ferritpreise, F301 als Sicherungseinsatz

Co-Authored-By: Claude Opus 5 <noreply@anthropic.com>
Parts:
- removed F301: Schurter 0034.3127, symbol Device:Fuse
- removed FB303, FB304, FB305, FB306, FB307: 330R@100MHz, Inductor_SMD:L_0805_2012Metric, symbol aa_MyParts:L_Ferrite_MH2029-601Y
- removed R300: 2mR CRF2010-FZ-R002ELF, Resistor_SMD:R_2010_5025Metric, symbol Device:R
- removed R310: 2R49, Resistor_SMD:R_0603_1608Metric, symbol Device:R
- added F301: 10A 250VAC, symbol aa_MyParts:F_0034.3127
- added FB303, FB304, FB306, FB307: 330R@100MHz, Inductor_SMD:L_0402_1005Metric, symbol aa_MyParts:L_Ferrite_BLM15EX331SN1D
- added R300: 2mR, Resistor_SMD:R_2010_5025Metric, symbol aa_MyParts:R_CRF2010-FZ-R002ELF
- added R318: 47k, Resistor_SMD:R_0603_1608Metric, symbol Device:R
- C300: Distributor 1 Order Number 710-890334023023CS -> 710-890334023023CS
- C302: Distributor 1 Order Number 710-860010673012 -> 710-860010673012
- renumbered PS300 to U307
Connections:
- net GND1 is gone; now on net GND: C307.2, C308.2, C311.2, U300.10 (GND1), U300.7 (LF)
- net +3V3: now also FB306.2, FB307.2
- net +3V3_ISO: now also FB303.1
- net GND: no longer J302.4 (Pin_4)
- net GND2_ISO: now also FB304.2
- net GND_ISO: now also FB304.1
- net PIN_N: now also R300.1
- net VDD: now also FB307.1, R318.2; no longer U300.5 (EN)
- net VIO: now also FB306.1
- net V_ISO_OUT: now also FB303.2
- net at FB302.2, K300.8: now also R300.2
- net PIN_L_SWITCHED: now reaches J301.1 (Pin_1), J301.2 (Pin_2), K300.2
- net PIN_N_SWITCHED: now reaches J301.3 (Pin_3), J301.4 (Pin_4), K300.6
- net Earth renamed PIN_PE
- new net ISO_EN: J302.4 (Pin_4), R318.1, U300.5 (EN)
- no-connect marks 15 -> 17
Other:
- note added: "CLEARANCE & CREEPAGE -- I/O BOARD 230V Basis: IEC 60664-1, 250 VAC working voltage, OVC II, pollution degree 2 (sealed IP64 enclosure), material group IIIa. Design minima in mm, valid for clearance AND creepage, on both layers. | NET same | NET opp. | ISO isl. | SELV ------------------|----------|----------|----------|------- NET same pole | 0.5 | 3.0 | 0.5 | 8.0 NET opposite | | 0.5 | 3.0 | 8.0 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"
- note added: "GAIN = 1"
- note added: "GAIN = 16"
- note added: "NET CLASS TRACK WIDTHS -- I/O BOARD 230V 2 layers, 70 um (2 oz), FR4 1.6 mm. IPC-2221 outer layer, dT = 5 K. Net class | I max | Width | Via ------------|---------|--------|------ 230V_ext | 8.000 A | 4.0 mm | 5x D PE | 8.000 A | 4.0 mm | 5x D 230V_int | 0.500 A | 1.0 mm | 1x C 5V | 2.000 A | 1.0 mm | 2x C 24V | 0.500 A | 0.8 mm | 1x C 3V3 | 1.000 A | 0.5 mm | 1x C ISO_signals | 0.020 A | 0.4 mm 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"
- note added: "Provide cooling area"
- note added: "VIAS -- 20 um barrel plating, dT 5 K. "per via" is what one via carries. Derate by 0.7 in dense via fields. Via | Drill | Pad | Aspect | per via ----|--------|---------|--------|--------- A | 0.2 mm | 0.45 mm | 8:1 | 0.839 A B | 0.3 mm | 0.6 mm | 5.3:1 | 1.126 A C | 0.6 mm | 1.0 mm | 2.7:1 | 1.861 A D | 1.0 mm | 1.4 mm | 1.6:1 | 2.695 A"
- note removed: "250V 10AT"
- company: (none) -> FREILab Freiburg e.V.
- title: (none) -> Schematic I/O Board
- moved on the sheet: C303, J301
