File: hardware/projects/RFID_BOX/ECAD/IO_Board/IO_Board.kicad_sch (KiCad schematic)
At the start: 72 parts, among them J300 J_WAGO_2604-1103, J301 J_WAGO_2604-1103, J302 Conn_01x10_Pin, K300 T92S11D12-24, Q300 2N7002NXAKR, Q301 BSS84AK, Q302 2N7002NXAKR, U300 ISOW7721DFMR, U301 IRM-10-24, U302 MCP39F511A-E/MQ, U306 R-78K5.0-2.0, U307 AP2114H-3.3TRG1

Commit message: work on layout
Parts:
- added R319, R320: 0R, Resistor_SMD:R_0603_1608Metric, symbol Device:R
Connections:
- net PIN_L_SWITCHED: now also K300.6; no longer K300.2
- net PIN_N_SWITCHED: now also K300.2; no longer K300.6
- net UART_MCP2MCU_ISO: now also R319.2; no longer U302.12 (UART_TX)
- net UART_MCU2MCP_ISO: now also R320.2; no longer U302.4 (UART_RX)
- net PIN_N_SHUNT: now reaches FB302.2, R300.2
- net PIN_N_SHUNT: now also K300.4; no longer K300.8
- net PIN_L_SENSE: now reaches FB300.1, R303.1
- net PIN_L_DIV: now reaches R303.2, R304.1
- net AVDD: now reaches C322.1, C323.1, R307.2, U302.11 (AVDD)
- net PIN_L_nc: now reaches K300.7
- net PIN_N_nc: now reaches K300.3
- net PIN_L_CTRL_F: now reaches F302.2, L300.1
- net PIN_CTRL_L renamed PIN_L_CTRL
- net PIN_CTRL_N renamed PIN_N_CTRL
- net PIN_FUSED_L renamed PIN_L_FUSED
- net PIN_L_FUSED: now also K300.8; no longer K300.4
- new net: R319.1, U302.12 (UART_TX)
- new net: R320.1, U302.4 (UART_RX)
Other:
- note added: "CLEARANCE & CREEPAGE -- I/O BOARD 230V Master table, binding for layout and DRC rules. Basis: IEC 60664-1, 250 VAC working voltage, OVC II, pollution degree 2 (sealed IP64 enclosure), material group IIIa. Design minima in mm, valid for clearance AND creepage, on both layers. L / N = mains poles, ISO = measurement island (at N potential via NT300), SELV = everything else, PE = protective earth (ba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"
- note added: "Groups: L = PIN_L* N = PIN_N* ISO = ISO_signals PE = PE SELV = Signals, 5V, 24V, Default"
- note removed: "CLEARANCE & CREEPAGE -- I/O BOARD 230V Basis: IEC 60664-1, 250 VAC working voltage, OVC II, pollution degree 2 (sealed IP64 enclosure), material group IIIa. Design minima in mm, valid for clearance AND creepage, on both layers. | NET same | NET opp. | ISO isl. | SELV ------------------|----------|----------|----------|------- NET same pole | 0.5 | 3.0 | 0.5 | 8.0 NET opposite | | 0.5 | 3.0 | 8.0 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"
